Commit message: model additional collision volumes

File: cu_panda_description/robots/basic_setup.urdf.xacro (robot description, xacro)
@@ -58,3 +58,65 @@
     <origin xyz="0 0 0.026" rpy="0 0 0"/>
   </joint>
+  <link name="window_collider">
+    <collision>
+      <geometry>
+        <box size="1.0 0.2 1.5"/>
+      </geometry>
+      <origin xyz="0 0 0.0" rpy="0 0 0"/>
+    </collision>
+    <visual>
+      <geometry>
+        <box size="1.0 0.2 1.5"/>
+      </geometry>
+      <origin xyz="0 0 0.0" rpy="0 0 0"/>
+      <material name="virtualvolume">
+        <color rgba="0.3 0.3 0.3 0.1"/>
+      </material>
+    </visual>
+  </link>
+  <joint name="window_collider_joint" type="fixed">
+    <child link="window_collider"/>
+    <parent link="table"/>
+    <origin xyz="0 ${-1.074/2-0.1-0.15} ${1.5/2}" rpy="0 0 0"/>
+  </joint>
+  <link name="wall">
+    <collision>
+      <geometry>
+        <box size="0.1 2.0 1.5"/>
+      </geometry>
+      <origin xyz="0 0 0" rpy="0 0 0"/>
+    </collision>
+    <visual>
+      <geometry>
+        <box size="0.1 2.0 1.5"/>
+      </geometry>
+      <origin xyz="0 0 0" rpy="0 0 0"/>
+      <material name="lightgrey"/>
+    </visual>
+  </link>
+  <joint name="wall_joint" type="fixed">
+    <child link="wall"/>
+    <parent link="table"/>
+    <origin xyz="${-0.35-0.05-0.19} 0 0.75" rpy="0 0 0"/>
+  </joint>
+  <link name="behind_table_collider">
+    <collision>
+      <geometry>
+        <box size="0.19 1.7 ${0.08+0.026}"/>
+      </geometry>
+      <origin xyz="0 0 0" rpy="0 0 0"/>
+    </collision>
+    <visual>
+      <geometry>
+        <box size="0.19 1.7 ${0.08+0.026}"/>
+      </geometry>
+      <origin xyz="0 0 0" rpy="0 0 0"/>
+      <material name="lightgrey"/>
+    </visual>
+  </link>
+  <joint name="behind_table_collider_joint" type="fixed">
+    <child link="behind_table_collider"/>
+    <parent link="table"/>
+    <origin xyz="${-0.35-0.095} 0 ${0.026}" rpy="0 0 0"/>
+  </joint>
 </robot>

Commit message: include realsense
calibration set by hand in rviz. It seems accurate within 0.02m for now.

File: cu_panda_description/robots/basic_setup.urdf.xacro (robot description, xacro)
@@ -120,3 +120,16 @@
     <origin xyz="${-0.35-0.095} 0 ${0.026}" rpy="0 0 0"/>
   </joint>
+  <link name="realsense_link">
+    <collision>
+      <geometry>
+        <box size="0.1 0.2 0.08"/>
+      </geometry>
+      <origin xyz="0 0 0" rpy="0 0 0"/>
+    </collision>
+  </link>
+  <joint name="realsense_table_joint" type="fixed">
+    <child link="realsense_link"/>
+    <parent link="table"/>
+    <origin xyz="-0.34866 0.48523 0.34558" rpy="-2.9583 2.6983 2.2201"/>
+  </joint>
 </robot>

Commit message: integrate short fingertip models

File: cu_panda_description/robots/basic_setup.urdf.xacro (robot description, xacro)
@@ -1,4 +1,5 @@
 <?xml version="1.0"?>
 <robot xmlns:xacro="http://ros.org/wiki/xacro" name="cu_panda">
+  <xacro:arg name="with_shortfingertips" default="true"/>
   <xacro:include filename="$(find cu_panda_description)/urdf/franka_robot_no_tips.urdf.xacro"/>
   <xacro:franka_robot arm_id="panda"
@@ -133,3 +134,41 @@
     <origin xyz="-0.34866 0.48523 0.34558" rpy="-2.9583 2.6983 2.2201"/>
   </joint>
+  <xacro:macro name="fingertip" params="side *origin">
+      <link name="panda_${side}tip_body">
+      <visual>
+        <origin xyz="0 0 0" rpy="0 0 0"/>
+        <geometry>
+          <mesh filename="package://cu_panda_description/meshes/panda_short_finger_adapted.stl" />
+        </geometry>
+        <material name="darkgrey">
+          <color rgba="0.1 0.1 0.1 1.0"/>
+        </material>
+      </visual>
+      <collision>
+        <origin xyz="0 -0.0045 ${(0.029+0.009)/2-0.009}" rpy="0 0 0"/>
+        <geometry>
+          <box size="0.02 0.009 ${0.029+0.009}"/>
+        </geometry>
+      </collision>
+    </link>
+    <joint name="panda_${side}tip_joint" type="fixed">
+      <parent link="panda_${side}tip_mount" />
+      <child link="panda_${side}tip_body" />
+      <xacro:insert_block name="origin"/>
+    </joint>
+    <link name="panda_${side}tip"/>
+    <joint name="panda_${side}tip_fixed_joint" type="fixed">
+      <parent link="panda_${side}tip_body" />
+      <child link="panda_${side}tip" />
+      <origin xyz="0 -0.009 0.019" rpy="0 0 0"/>
+    </joint>
+  </xacro:macro>
+  <xacro:if value="$(arg with_shortfingertips)">
+    <xacro:fingertip side="left">
+      <origin xyz="0.0 0.0 0.0" rpy="0 0 0"/>
+    </xacro:fingertip>
+    <xacro:fingertip side="right">
+      <origin xyz="0.0 0.0 0.0" rpy="0 0 ${tau/2}"/>
+    </xacro:fingertip>
+  </xacro:if>
 </robot>

File: cu_panda_description/urdf/franka_hand_no_tips.urdf.xacro (robot description, xacro)
@@ -50,9 +50,9 @@
         </geometry>
       </collision>
-      <!-- rubber tip with which to grasp -->
+      <!-- mounting segment for tips -->
       <collision>
-        <origin xyz="0 7.58e-3 45.25e-3" rpy="0 0 0" />
+        <origin xyz="0 14.5e-3 45.25e-3" rpy="0 0 0" />
         <geometry>
-          <box size="17.5e-3 15.2e-3 18.5e-3" />
+          <box size="17.5e-3 10.2e-3 18.5e-3" />
         </geometry>
       </collision>
@@ -61,4 +61,10 @@
       </xacro:if>
     </link>
+    <link name="${arm_id}_lefttip_mount"/>
+    <joint name="${arm_id}_lefttip_mount_joint" type="fixed">
+      <parent link="${arm_id}_leftfinger" />
+      <child link="${arm_id}_lefttip_mount" />
+      <origin xyz="0.0 0.01 0.045" rpy="0 0 0"/>
+    </joint>
     <link name="${arm_id}_rightfinger">
       <visual>
@@ -89,9 +95,9 @@
         </geometry>
       </collision>
-      <!-- rubber tip with which to grasp -->
+      <!-- mounting segment for tips -->
       <collision>
-        <origin xyz="0 -7.58e-3 45.25e-3" rpy="0 0 0" />
+        <origin xyz="0 -14.5e-3 45.25e-3" rpy="0 0 0" />
         <geometry>
-          <box size="17.5e-3 15.2e-3 18.5e-3" />
+          <box size="17.5e-3 10.2e-3 18.5e-3" />
         </geometry>
       </collision>
@@ -100,4 +106,10 @@
       </xacro:if>
     </link>
+    <link name="${arm_id}_righttip_mount"/>
+    <joint name="${arm_id}_righttip_mount_joint" type="fixed">
+      <parent link="${arm_id}_rightfinger" />
+      <child link="${arm_id}_righttip_mount" />
+      <origin xyz="0.0 -0.01 0.045" rpy="0 0 0"/>
+    </joint>
     <joint name="${arm_id}_finger_joint1" type="prismatic">
       <parent link="${arm_id}_hand" />

Commit message: adjust distance to wall
it appears the (rather heavy) table moved over time.
Now we add 6cm safety padding to the physical wall location.

File: cu_panda_description/robots/basic_setup.urdf.xacro (robot description, xacro)
@@ -99,5 +99,5 @@
     <child link="wall"/>
     <parent link="table"/>
-    <origin xyz="${-0.35-0.05-0.19} 0 0.75" rpy="0 0 0"/>
+    <origin xyz="${-0.35-0.05-0.10} 0 0.75" rpy="0 0 0"/>
   </joint>
   <link name="behind_table_collider">

Commit message: reduced mounting plate size by 2 mm, to reduce the diffrence between how the robot is shown to touch the table in rviz and real life

File: cu_panda_description/robots/basic_setup.urdf.xacro (robot description, xacro)
@@ -12,5 +12,5 @@
     <visual>
       <geometry>
-        <box size="0.32 0.216 0.026"/>
+        <box size="0.32 0.216 0.024"/>
       </geometry>
       <material name="lightblack">
@@ -21,5 +21,5 @@
     <collision>
       <geometry>
-        <box size="0.32 0.216 0.034"/>
+        <box size="0.32 0.216 0.032"/>
       </geometry>
       <origin xyz="0 0 0.017" rpy="0 0 0"/>
@@ -29,5 +29,5 @@
     <child link="panda_link0"/>
     <parent link="panda_mounting_plate"/>
-    <origin xyz="0.033 0 0.026" rpy="0 0 0"/>
+    <origin xyz="0.033 0 0.024" rpy="0 0 0"/>
   </joint>
   <link name="table">

Commit message: recalibrated camera

File: cu_panda_description/robots/basic_setup.urdf.xacro (robot description, xacro)
@@ -51,5 +51,5 @@
     <child link="panda_mounting_plate"/>
     <parent link="table"/>
-    <origin xyz="${-0.35+0.16} ${-0.537+0.04+0.108} 0.026" rpy="0 0 0"/>
+    <origin xyz="${-0.35+0.16} ${-0.537+0.04+0.108} 0.027" rpy="0 0 0"/>
   </joint>
   <link name="table_top"/>
@@ -57,5 +57,5 @@
     <child link="table_top"/>
     <parent link="table"/>
-    <origin xyz="0 0 0.026" rpy="0 0 0"/>
+    <origin xyz="0 0 0.027" rpy="0 0 0"/>
   </joint>
   <link name="window_collider">
@@ -121,4 +121,5 @@
     <origin xyz="${-0.35-0.095} 0 ${0.026}" rpy="0 0 0"/>
   </joint>
+ <!-- # -0.353; 0.48923; 0.3458 -->
   <link name="realsense_link">
     <collision>
@@ -132,5 +133,5 @@
     <child link="realsense_link"/>
     <parent link="table"/>
-    <origin xyz="-0.34866 0.48523 0.34558" rpy="-2.9583 2.6983 2.2201"/>
+    <origin xyz="-0.360 0.490 0.342" rpy="0.192 0.436 -0.908"/>
   </joint>
   <xacro:macro name="fingertip" params="side *origin">
